Commit message: Add Makefile and simulation parameter support in launch/xacro, update Dockerfile

File: robot_description/urdf/robot.urdf.xacro (robot description, xacro)
@@ -1,44 +1,6 @@
 <?xml version="1.0"?>
 <robot xmlns:xacro="http://ros.org/wiki/xacro" name="template_robot">
-  <!-- Reference point on the ground -->
-  <link name="base_footprint"/>
-  <!-- Base body (blue box) -->
-  <link name="base_link">
-    <visual>
-      <geometry>
-        <box size="0.2 0.2 0.2"/>
-      </geometry>
-      <material name="blue">
-        <color rgba="0.0 0.0 1.0 1.0"/>
-      </material>
-    </visual>
-  </link>
-  <!-- Attach base_link to base_footprint (so the robot sits on the ground) -->
-  <joint name="base_footprint_to_base_link" type="fixed">
-    <parent link="base_footprint"/>
-    <child link="base_link"/>
-    <origin xyz="0 0 0.1" rpy="0 0 0"/>
-  </joint>
-  <!-- A smaller link (green box) -->
-  <link name="moving_link">
-    <visual>
-      <geometry>
-        <box size="0.1 0.1 0.1"/>
-      </geometry>
-      <material name="green">
-        <color rgba="0.0 1.0 0.0 1.0"/>
-      </material>
-    </visual>
-  </link>
-  <!-- Movable joint: rotates the green box around Z axis -->
-  <joint name="base_to_moving_joint" type="revolute">
-    <parent link="base_link"/>
-    <child link="moving_link"/>
-    <!-- Place the moving_link slightly to the side and above the base -->
-    <origin xyz="0 0 0.15" rpy="0 0 0"/>
-    <!-- Rotation axis Z -->
-    <axis xyz="0 0 1"/>
-    <!-- Limits: +/- 90 degrees -->
-    <limit effort="10" velocity="1.0" lower="-1.57" upper="1.57"/>
-  </joint>
+  <xacro:include filename="$(find robot_description)/urdf/robot_arguments.xacro" />
+  <xacro:include filename="$(find robot_description)/urdf/blue_box.xacro" />
+  <xacro:include filename="$(find robot_description)/urdf/green_box.xacro" />
 </robot>
