Commit message: Add collision and inertial

File: robot_description/urdf/blue_box.xacro (robot description, xacro)
@@ -13,6 +13,14 @@
             </material>
         </visual>
+        <collision>
+            <geometry>
+                <box size="0.2 0.2 0.2" />
+            </geometry>
+        </collision>
+        <inertial>
+            <mass value="1" />
+            <inertia ixx="0.01" iyy="0.01" izz="0.01" ixy="0" ixz="0" iyz="0" />
+        </inertial>
     </link>
-    <!-- Attach base_link to base_footprint (so the robot sits on the ground) -->
     <joint name="base_footprint_to_base_link" type="fixed">
         <parent link="base_footprint" />

File: robot_description/urdf/green_box.xacro (robot description, xacro)
@@ -11,4 +11,13 @@
                 </material>
             </visual>
+            <collision>
+                <geometry>
+                    <box size="0.1 0.1 0.1" />
+                </geometry>
+            </collision>
+            <inertial>
+                <mass value="1" />
+                <inertia ixx="0.01" iyy="0.01" izz="0.01" ixy="0" ixz="0" iyz="0" />
+            </inertial>
         </link>
         <!-- Movable joint: rotates the green box around Z axis -->
