Commit message: Fix urdf mesh path

File: robot_description/urdf/realsence_d435_macro.xacro (robot description, xacro)
@@ -37,5 +37,5 @@
             rpy="${M_PI/2} 0 ${M_PI/2}" />
           <geometry>
-            <mesh filename="file://$(find robot_description)/meshes/realsence_d435.dae" />
+            <mesh filename="package://robot_description/meshes/realsence_d435.dae" />
           </geometry>
         </xacro:if>

File: robot_description/urdf/robot_core.xacro (robot description, xacro)
@@ -6,5 +6,5 @@
             <origin xyz="-0.032 0 0.0" rpy="0 0 0" />
             <geometry>
-                <mesh filename="file://$(find robot_description)/meshes/base.stl"
+                <mesh filename="package://robot_description/meshes/base.stl"
                     scale="0.001 0.001 0.001" />
             </geometry>
@@ -14,5 +14,5 @@
             <origin xyz="-0.032 0 0.000" rpy="0 0 0" />
             <geometry>
-                <mesh filename="file://$(find robot_description)/meshes/base.stl"
+                <mesh filename="package://robot_description/meshes/base.stl"
                     scale="0.001 0.001 0.001" />
             </geometry>
@@ -42,5 +42,5 @@
             <origin xyz="0 0 0" rpy="1.57 0 0" />
             <geometry>
-                <mesh filename="file://$(find robot_description)/meshes/left_wheel.stl"
+                <mesh filename="package://robot_description/meshes/left_wheel.stl"
                     scale="0.001 0.001 0.001" />
             </geometry>
@@ -72,5 +72,5 @@
             <origin xyz="0 0 0" rpy="1.57 0 0" />
             <geometry>
-                <mesh filename="file://$(find robot_description)/meshes/right_wheel.stl"
+                <mesh filename="package://robot_description/meshes/right_wheel.stl"
                     scale="0.001 0.001 0.001" />
             </geometry>

File: robot_description/urdf/rplidar_a2m8.xacro (robot description, xacro)
@@ -11,5 +11,5 @@
                 <origin xyz="0.005 0.03 -0.031" rpy="0 0 2.8" />
                 <geometry>
-                    <mesh filename="file://$(find robot_description)/meshes/rplidar_a2m8.stl"
+                    <mesh filename="package://robot_description/meshes/rplidar_a2m8.stl"
                         scale="0.001 0.001 0.001" />
                 </geometry>

Commit message: Add env, fix mesh path

File: robot_description/urdf/realsence_d435_macro.xacro (robot description, xacro)
@@ -37,5 +37,5 @@
             rpy="${M_PI/2} 0 ${M_PI/2}" />
           <geometry>
-            <mesh filename="package://robot_description/meshes/realsence_d435.dae" />
+            <mesh filename="file://$(find robot_description)/meshes/realsence_d435.dae" />
           </geometry>
         </xacro:if>

File: robot_description/urdf/robot_core.xacro (robot description, xacro)
@@ -6,5 +6,5 @@
             <origin xyz="-0.032 0 0.0" rpy="0 0 0" />
             <geometry>
-                <mesh filename="package://robot_description/meshes/base.stl"
+                <mesh filename="file://$(find robot_description)/meshes/base.stl"
                     scale="0.001 0.001 0.001" />
             </geometry>
@@ -14,5 +14,5 @@
             <origin xyz="-0.032 0 0.000" rpy="0 0 0" />
             <geometry>
-                <mesh filename="package://robot_description/meshes/base.stl"
+                <mesh filename="file://$(find robot_description)/meshes/base.stl"
                     scale="0.001 0.001 0.001" />
             </geometry>
@@ -42,5 +42,5 @@
             <origin xyz="0 0 0" rpy="1.57 0 0" />
             <geometry>
-                <mesh filename="package://robot_description/meshes/left_wheel.stl"
+                <mesh filename="file://$(find robot_description)/meshes/left_wheel.stl"
                     scale="0.001 0.001 0.001" />
             </geometry>
@@ -72,5 +72,5 @@
             <origin xyz="0 0 0" rpy="1.57 0 0" />
             <geometry>
-                <mesh filename="package://robot_description/meshes/right_wheel.stl"
+                <mesh filename="file://$(find robot_description)/meshes/right_wheel.stl"
                     scale="0.001 0.001 0.001" />
             </geometry>

File: robot_description/urdf/rplidar_a2m8.xacro (robot description, xacro)
@@ -11,5 +11,5 @@
                 <origin xyz="0.005 0.03 -0.031" rpy="0 0 2.8" />
                 <geometry>
-                    <mesh filename="package://robot_description/meshes/rplidar_a2m8.stl"
+                    <mesh filename="file://$(find robot_description)/meshes/rplidar_a2m8.stl"
                         scale="0.001 0.001 0.001" />
                 </geometry>
